File: backplane.kicad_sch (KiCad schematic)
At the start: 49 parts, among them J1 DIN41612_02x32_AC, J10 DIN41612_02x32_AC, J11 DIN41612_02x32_AC, J12 Conn_01x04, J13 Conn_01x03, J14 Conn_01x03, J15 Conn_01x03, J16 Conn_01x03, J17 Conn_01x03, J18 Conn_01x03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

Commit message: kicad 10
Other:
- title: Backplane -> LaserRackBoars Backplane
